Commit message: fix omega when tracking a stationary point

File: src/four_wheel_drive/robot_model/xacro/smartcar_sim.xacro (robot description, xacro)
@@ -263,24 +263,4 @@
 		</actuator>
 	</transmission>
-	<transmission name="right_front_wheel_joint_trans">
-		<type>transmission_interface/SimpleTransmission</type>
-		<joint name="right_front_wheel_to_bridge" >
-			<hardwareInterface>hardware_interface/VelocityJointInterface</hardwareInterface>
-		</joint>
-		<actuator name="right_front_wheel_joint_motor">
-			<hardwareInterface>hardware_interface/VelocityJointInterface</hardwareInterface>
-			<mechanicalReduction>1</mechanicalReduction>
-		</actuator>
-	</transmission>
-	<transmission name="left_front_wheel_joint_trans">
-		<type>transmission_interface/SimpleTransmission</type>
-		<joint name="left_front_wheel_to_bridge" >
-			<hardwareInterface>hardware_interface/VelocityJointInterface</hardwareInterface>
-		</joint>
-		<actuator name="left_front_wheel_joint_motor">
-			<hardwareInterface>hardware_interface/VelocityJointInterface</hardwareInterface>
-			<mechanicalReduction>1</mechanicalReduction>
-		</actuator>
-	</transmission>
 	<!-- Friction Parametres -->
 <!--
